Commit message: need to write a local controller

File: mecanum_sim/urdf/mecanum.xacro (robot description, xacro)
@@ -200,5 +200,5 @@
   <joint name="camera_joint2" type="fixed">
     <axis xyz="0 1 0" />
-    <origin xyz="${camera_link2} 0 0.5" rpy="0 0.785 0"/>
+    <origin xyz="-0.05 0 0.5" rpy="0 0.785 0"/>
     <parent link="base_link"/>
     <child link="camera_link2"/>

Commit message: localization test

File: mecanum_sim/urdf/mecanum.xacro (robot description, xacro)
@@ -3,6 +3,6 @@
   <!-- include gazebo plugins -->
   <xacro:include filename="$(find mecanum_sim)/urdf/mecanum.gazebo" />
-  <xacro:property name="base_width" value="0.5" />   <!-- 14.5 in -->
-  <xacro:property name="base_length" value="0.5" />  <!-- 21 5/8 in -->
+  <xacro:property name="base_width" value="0.3476" />   <!-- 14.5 in -->
+  <xacro:property name="base_length" value="0.4" />  <!-- 21 5/8 in -->
   <xacro:property name="base_height" value="0.0635" />   <!-- 2.5 in  -->
   <xacro:property name="wheel_radius" value="0.1016" /> <!-- 4.0 in  -->
@@ -173,5 +173,5 @@
   <joint name="camera_joint1" type="fixed">
     <axis xyz="0 1 0" />
-    <origin xyz="${camera_link1} 0 0.7" rpy="0 0 0"/>
+    <origin xyz="-0.05 0 0.7" rpy="0 0 0"/>
     <parent link="base_link"/>
     <child link="camera_link1"/>
